Commit message: finalizing xacro.

File: urdf/omniveyor.gazebo.xacro (robot description, xacro)
@@ -1,4 +1,5 @@
 <?xml version="1.0" ?>
 <robot name="omniveyor" xmlns:xacro="http://www.ros.org/wiki/xacro">
+  <xacro:arg name="gpu_ray_tracing" default="true"/>
   <xacro:property name="steerAxisX" value="0.2074" />
   <xacro:property name="steerAxisY" value="0.2074" />
@@ -117,6 +118,5 @@
     <material>Gazebo/DarkGrey</material>
   </gazebo>
-  <gazebo reference="laser">
-      <sensor name="laser" type="gpu_ray">
+  <xacro:property name="lidar_params">
         <pose>0 0 0 0 -0 0</pose>
         <ray>
@@ -140,12 +140,27 @@
           <stddev>0.005</stddev>
         </noise>
+        <always_on>1</always_on>
+        <update_rate>40</update_rate>
+        <visualize>true</visualize>
+  </xacro:property>
+  <gazebo reference="laser">
+  <xacro:if value="$(arg gpu_ray_tracing)">
+      <sensor name="laser" type="gpu_ray">
+        <xacro:insert_block name="lidar_params"/>
         <plugin name="gazebo_ros_head_hokuyo_controller" filename="libgazebo_ros_gpu_laser.so">
           <topicName>scan</topicName>
           <frameName>laser</frameName>
         </plugin>
-        <always_on>1</always_on>
-        <update_rate>40</update_rate>
-        <visualize>true</visualize>
-      </sensor>
+      </sensor>
+  </xacro:if>
+  <xacro:unless value="$(arg gpu_ray_tracing)">
+      <sensor name="laser" type="ray">
+        <xacro:insert_block name="lidar_params"/>
+        <plugin name="gazebo_ros_head_hokuyo_controller" filename="libgazebo_ros_laser.so">
+          <topicName>scan</topicName>
+          <frameName>laser</frameName>
+        </plugin>
+      </sensor>
+  </xacro:unless>
   </gazebo>
   <gazebo reference="cam_d1_link">
@@ -175,6 +190,6 @@
           <horizontal_fov>1.204</horizontal_fov>
           <image>
-            <width>1280</width>
-            <height>720</height>
+            <width>848</width>
+            <height>480</height>
             <format>R8G8B8</format>
           </image>
@@ -239,6 +254,6 @@
           <horizontal_fov>1.204</horizontal_fov>
           <image>
-            <width>1280</width>
-            <height>720</height>
+            <width>848</width>
+            <height>480</height>
             <format>R8G8B8</format>
           </image>

File: urdf/omniveyor.urdf.xacro (robot description, xacro)
@@ -2,4 +2,5 @@
 <robot name="omniveyor" xmlns:xacro="http://www.ros.org/wiki/xacro">
   <xacro:arg name="gazebo" default="false"/>
+  <xacro:arg name="gpu_ray_tracing" default="true"/>
   <xacro:include filename="omniveyor.materials.xacro"/>
   <xacro:if value="$(arg gazebo)">
@@ -106,5 +107,5 @@
     </inertial>
     <collision>
-      <origin xyz="-0.3752 0.3381 0.032" rpy="${-pi/2} 0 0"/>
+      <origin xyz="-0.3752 0.3381 0.032" rpy="${pi/2} 0 0"/>
       <geometry>
         <mesh filename="package://omniveyor_common/meshes/OV_Shell.STL"
@@ -113,5 +114,5 @@
     </collision>
     <visual>
-      <origin xyz="-0.3752 0.3381 0.032" rpy="${-pi/2} 0 0"/>
+      <origin xyz="-0.3752 0.3381 0.032" rpy="${pi/2} 0 0"/>
       <geometry>
         <mesh filename="package://omniveyor_common/meshes/OV_Shell.STL"

Commit message: compatibility with full-stack realSense simulation

File: urdf/omniveyor.gazebo.xacro (robot description, xacro)
@@ -1,5 +1,7 @@
 <?xml version="1.0" ?>
-<robot name="omniveyor" xmlns:xacro="http://www.ros.org/wiki/xacro">
+<robot xmlns:xacro="http://www.ros.org/wiki/xacro">
   <xacro:arg name="gpu_ray_tracing" default="true"/>
+  <xacro:property name="accurateRealsense" value="$(find omniveyor_gazebo_world)" />
+  <xacro:property name="accurateRrealsensePlugin" value="$(find realsense_ros_gazebo)" />
   <xacro:property name="steerAxisX" value="0.2074" />
   <xacro:property name="steerAxisY" value="0.2074" />
@@ -103,4 +105,5 @@
   <xacro:pcv_assembly prefix="RL"/>
   <xacro:pcv_assembly prefix="RR"/>
+  <xacro:unless value="${accurateRealsense != '' and accurateRrealsensePlugin != ''}">
   <link name="cam_d1_depth_link"/>
   <link name="cam_d2_depth_link"/>
@@ -115,4 +118,5 @@
     <origin xyz="0 0 0" rpy="${-pi/2} 0 ${-pi/2}" />
   </joint>
+  </xacro:unless>
   <gazebo reference="base_link">
     <material>Gazebo/DarkGrey</material>
@@ -164,4 +168,5 @@
   </xacro:unless>
   </gazebo>
+  <xacro:unless value="${accurateRealsense != '' and accurateRrealsensePlugin != ''}">
   <gazebo reference="cam_d1_link">
       <sensor name="imu_sensor" type="imu">
@@ -311,4 +316,5 @@
     </sensor>
   </gazebo>
+  </xacro:unless>
   <gazebo>
     <plugin filename="libOmniVeyorPlugin_ROS.so" name="omniveyor_simulator"/>

File: urdf/omniveyor.urdf.xacro (robot description, xacro)
@@ -3,4 +3,5 @@
   <xacro:arg name="gazebo" default="false"/>
   <xacro:arg name="gpu_ray_tracing" default="true"/>
+  <xacro:arg name="simulate_accurate_realsense_cameras" default="true"/>
   <xacro:include filename="omniveyor.materials.xacro"/>
   <xacro:if value="$(arg gazebo)">
@@ -9,4 +10,68 @@
     <xacro:include filename="omniveyor.gazebo.xacro"/>
   </xacro:if>
+  <!--geometric center of omniveyor (on-ground)-->
+  <link name="base_link">
+  <xacro:if value="$(arg gazebo)">
+    <inertial>
+      <origin xyz="0 0 0.192" rpy="0 0 0"/>
+      <mass value="29.82"/>
+      <inertia ixx="1.209698" ixy="0" ixz="0"
+          iyy="1.209698" iyz="0" izz="1.910468"/>
+    </inertial>
+    <collision>
+      <origin xyz="-0.3752 0.3381 0.032" rpy="${pi/2} 0 0"/>
+      <geometry>
+        <mesh filename="package://omniveyor_common/meshes/OV_Shell.STL"
+              scale="0.001 0.001 0.001"/>
+      </geometry>
+    </collision>
+    <visual>
+      <origin xyz="-0.3752 0.3381 0.032" rpy="${pi/2} 0 0"/>
+      <geometry>
+        <mesh filename="package://omniveyor_common/meshes/OV_Shell.STL"
+              scale="0.001 0.001 0.001"/>
+      </geometry>
+      <material name="grey"/>
+    </visual>
+  </xacro:if>
+  </link>
+  <!--Hokuyo 20LX-->
+  <link name="laser">
+  <xacro:if value="$(arg gazebo)">
+    <inertial>
+      <mass value="0.1"/>
+      <inertia ixx="0.01" ixy="0" ixz="0"
+               iyy="0.01" iyz="0" izz="0.01"/>
+    </inertial>
+    <visual name="visual">
+      <origin xyz="0 0 -0.0175" rpy="0 0 0"/>
+      <geometry>
+        <mesh filename="package://omniveyor_common/meshes/hokuyo.dae"/>
+      </geometry>
+    </visual>
+    <collision name="collision-base">
+      <origin xyz="0 0 -0.032" rpy="0 0 0"/>
+      <geometry>
+        <box size="0.05 0.05 0.041"/>
+      </geometry>
+    </collision>
+    <collision name="collision-top">
+      <origin xyz="0 0 0.003" rpy="0 0 0"/>
+      <geometry>
+        <cylinder radius="0.021" length="0.029"/>
+      </geometry>
+    </collision>
+  </xacro:if>
+  </link>
+  <joint name="laser_joint" type="fixed">
+  <!--laser connector from bottom (on-ground) center of omniveyor-->
+    <parent link="base_link" />
+    <child link="laser" />
+    <origin xyz="0.27 0 0.10" rpy="0 0 0" />
+  </joint>
+  <xacro:property name="accurateRealsense" value="$(find omniveyor_gazebo_world)" />
+  <xacro:property name="accurateRrealsensePlugin" value="$(find realsense_ros_gazebo)" />
+  <xacro:property name="gazebo_property" value="$(arg gazebo)"/>
+  <xacro:unless value="${accurateRealsense != '' and accurateRrealsensePlugin != '' and gazebo_property}">
   <!--tracking camera-->
   <link name="cam_t1_pose_frame">
@@ -69,64 +134,4 @@
   </xacro:if>
   </link>
-  <!--Hokuyo 20LX-->
-  <link name="laser">
-  <xacro:if value="$(arg gazebo)">
-    <inertial>
-      <mass value="0.1"/>
-      <inertia ixx="0.01" ixy="0" ixz="0"
-               iyy="0.01" iyz="0" izz="0.01"/>
-    </inertial>
-    <visual name="visual">
-      <origin xyz="0 0 -0.0175" rpy="0 0 0"/>
-      <geometry>
-        <mesh filename="package://omniveyor_common/meshes/hokuyo.dae"/>
-      </geometry>
-    </visual>
-    <collision name="collision-base">
-      <origin xyz="0 0 -0.032" rpy="0 0 0"/>
-      <geometry>
-        <box size="0.05 0.05 0.041"/>
-      </geometry>
-    </collision>
-    <collision name="collision-top">
-      <origin xyz="0 0 0.003" rpy="0 0 0"/>
-      <geometry>
-        <cylinder radius="0.021" length="0.029"/>
-      </geometry>
-    </collision>
-  </xacro:if>
-  </link>
-  <!--geometric center of omniveyor (on-ground)-->
-  <link name="base_link">
-  <xacro:if value="$(arg gazebo)">
-    <inertial>
-      <origin xyz="0 0 0.192" rpy="0 0 0"/>
-      <mass value="29.82"/>
-      <inertia ixx="1.209698" ixy="0" ixz="0"
-          iyy="1.209698" iyz="0" izz="1.910468"/>
-    </inertial>
-    <collision>
-      <origin xyz="-0.3752 0.3381 0.032" rpy="${pi/2} 0 0"/>
-      <geometry>
-        <mesh filename="package://omniveyor_common/meshes/OV_Shell.STL"
-              scale="0.001 0.001 0.001"/>
-      </geometry>
-    </collision>
-    <visual>
-      <origin xyz="-0.3752 0.3381 0.032" rpy="${pi/2} 0 0"/>
-      <geometry>
-        <mesh filename="package://omniveyor_common/meshes/OV_Shell.STL"
-              scale="0.001 0.001 0.001"/>
-      </geometry>
-      <material name="grey"/>
-    </visual>
-  </xacro:if>
-  </link>
-  <joint name="laser_joint" type="fixed">
-  <!--laser connector from bottom (on-ground) center of omniveyor-->
-    <parent link="base_link" />
-    <child link="laser" />
-    <origin xyz="0.27 0 0.10" rpy="0 0 0" />
-  </joint>
   <joint name="front_t265_joint" type="fixed">
   <!--front tracking camera connector from bottom (on-ground) center of omniveyor-->
@@ -147,3 +152,7 @@
     <origin xyz="-0.285 -0.08 0.37" rpy="0 0.04 ${pi}" />
   </joint>
+  </xacro:unless>
+  <xacro:if value="${accurateRealsense != '' and accurateRrealsensePlugin != '' and gazebo_property}">
+    <xacro:include filename="$(find omniveyor_gazebo_world)/launch/realsense_accurate_setup.gazebo.xacro"/>
+  </xacro:if>
 </robot>
