Commit message: unified all topics and sensor behaviors. Debugged spawning multiple robots

File: urdf/omniveyor.gazebo.xacro (robot description, xacro)
@@ -2,6 +2,4 @@
 <robot xmlns:xacro="http://www.ros.org/wiki/xacro">
   <xacro:arg name="gpu_ray_tracing" default="true"/>
-  <xacro:property name="accurateRealsense" value="$(find omniveyor_gazebo_world)" />
-  <xacro:property name="accurateRrealsensePlugin" value="$(find realsense_ros_gazebo)" />
   <xacro:property name="steerAxisX" value="0.2074" />
   <xacro:property name="steerAxisY" value="0.2074" />
@@ -105,23 +103,9 @@
   <xacro:pcv_assembly prefix="RL"/>
   <xacro:pcv_assembly prefix="RR"/>
-  <xacro:unless value="${accurateRealsense != '' and accurateRrealsensePlugin != ''}">
-  <link name="cam_d1_depth_link"/>
-  <link name="cam_d2_depth_link"/>
-  <joint name="cam_d1_depth_conversion" type="fixed">
-    <parent link="cam_d1_link" />
-    <child link="cam_d1_depth_link" />
-    <origin xyz="0 0 0" rpy="${-pi/2} 0 ${-pi/2}" />
-  </joint>
-  <joint name="cam_d2_depth_conversion" type="fixed">
-    <parent link="cam_d2_link" />
-    <child link="cam_d2_depth_link" />
-    <origin xyz="0 0 0" rpy="${-pi/2} 0 ${-pi/2}" />
-  </joint>
-  </xacro:unless>
-  <gazebo reference="base_link">
+  <gazebo reference="chassis">
     <material>Gazebo/DarkGrey</material>
   </gazebo>
   <xacro:property name="lidar_params">
-        <pose>0 0 0 0 -0 0</pose>
+        <pose>0 0 0 0 0 0</pose>
         <ray>
           <scan>
@@ -138,10 +122,10 @@
             <resolution>0.01</resolution>
           </range>
+          <noise>
+            <type>gaussian</type>
+            <mean>0.0</mean>
+            <stddev>0.01</stddev>
+          </noise>
         </ray>
-        <noise>
-          <type>gaussian</type>
-          <mean>0.0</mean>
-          <stddev>0.005</stddev>
-        </noise>
         <always_on>1</always_on>
         <update_rate>40</update_rate>
@@ -168,153 +152,4 @@
   </xacro:unless>
   </gazebo>
-  <xacro:unless value="${accurateRealsense != '' and accurateRrealsensePlugin != ''}">
-  <gazebo reference="cam_d1_link">
-      <sensor name="imu_sensor" type="imu">
-        <gravity>true</gravity>
-        <always_on>true</always_on>
-        <update_rate>100</update_rate>
-        <visualize>true</visualize>
-        <plugin filename="libgazebo_ros_imu_sensor.so" name="imu_plugin">
-          <topicName>/cam_d1/imu</topicName>
-          <bodyName>cam_d1_link</bodyName>
-          <updateRateHZ>0.0</updateRateHZ>
-          <gaussianNoise>0.002</gaussianNoise>
-          <xyzOffset>0 0 0</xyzOffset>
-          <rpyOffset>0 0 0</rpyOffset>
-          <frameName>cam_d1_link</frameName>
-          <initialOrientationAsReference>false</initialOrientationAsReference>
-        </plugin>
-        <pose>0 0 0 0 0 0</pose>
-      </sensor>
-      <sensor name="camera" type="depth">
-        <!--pose>0.001 -0.045 0.003 0 0 0</pose-->
-        <pose> 0 0 0 0 0 0 </pose>
-        <visualize>true</visualize>
-        <update_rate>15</update_rate>
-        <camera>
-          <horizontal_fov>1.204</horizontal_fov>
-          <image>
-            <width>848</width>
-            <height>480</height>
-            <format>R8G8B8</format>
-          </image>
-          <noise>
-            <type>gaussian</type>
-            <mean>0.0</mean>
-            <stddev>0.007</stddev>
-          </noise>
-        </camera>
-        <plugin name="camera_plugin" filename="libgazebo_ros_openni_kinect.so">
-          <baseline>0.2</baseline>
-          <alwaysOn>true</alwaysOn>
-          <!-- Keep this zero, update_rate in the parent <sensor> tag
-            will control the frame rate. -->
-          <updateRate>0.0</updateRate>
-          <cameraName>cam_d1</cameraName>
-          <imageTopicName>/cam_d1/color/image_raw</imageTopicName>
-          <cameraInfoTopicName>/cam_d1/color/camera_info</cameraInfoTopicName>
-          <depthImageTopicName>/cam_d1/depth/image_rect_raw</depthImageTopicName>
-          <depthImageCameraInfoTopicName>/cam_d1/depth/camera_info</depthImageCameraInfoTopicName>
-          <pointCloudTopicName>/cam_d1/depth/color/points</pointCloudTopicName>
-          <frameName>cam_d1_depth_link</frameName>
-          <pointCloudCutoff>0.3</pointCloudCutoff>
-          <pointCloudCutoffMax>8.0</pointCloudCutoffMax>
-          <distortionK1>0</distortionK1>
-          <distortionK2>0</distortionK2>
-          <distortionK3>0</distortionK3>
-          <distortionT1>0</distortionT1>
-          <distortionT2>0</distortionT2>
-          <CxPrime>0</CxPrime>
-          <Cx>0</Cx>
-          <Cy>0</Cy>
-          <focalLength>0</focalLength>
-          <hackBaseline>0</hackBaseline>
-        </plugin>
-      </sensor>
-  </gazebo>
-  <gazebo reference="cam_d2_link">
-      <sensor name="imu_sensor" type="imu">
-        <always_on>true</always_on>
-        <update_rate>100</update_rate>
-        <visualize>true</visualize>
-        <gravity>true</gravity>
-        <plugin filename="libgazebo_ros_imu_sensor.so" name="imu_plugin">
-          <topicName>/cam_d2/imu</topicName>
-          <bodyName>cam_d2_link</bodyName>
-          <updateRateHZ>0.0</updateRateHZ>
-          <gaussianNoise>0.002</gaussianNoise>
-          <xyzOffset>0 0 0</xyzOffset>
-          <rpyOffset>0 0 0</rpyOffset>
-          <frameName>cam_d2_link</frameName>
-          <initialOrientationAsReference>false</initialOrientationAsReference>
-        </plugin>
-        <pose>0 0 0 0 0 0</pose>
-      </sensor>
-      <sensor name="camera" type="depth">
-        <!--pose>0.001 -0.045 0.003 0 0 0</pose-->
-        <pose> 0 0 0 0 0 0 </pose>
-        <visualize>true</visualize>
-        <update_rate>15</update_rate>
-        <camera>
-          <horizontal_fov>1.204</horizontal_fov>
-          <image>
-            <width>848</width>
-            <height>480</height>
-            <format>R8G8B8</format>
-          </image>
-          <noise>
-            <type>gaussian</type>
-            <mean>0.0</mean>
-            <stddev>0.007</stddev>
-          </noise>
-        </camera>
-        <plugin name="camera_plugin" filename="libgazebo_ros_openni_kinect.so">
-          <baseline>0.2</baseline>
-          <alwaysOn>true</alwaysOn>
-          <!-- Keep this zero, update_rate in the parent <sensor> tag
-            will control the frame rate. -->
-          <updateRate>0.0</updateRate>
-          <cameraName>cam_d2</cameraName>
-          <imageTopicName>/cam_d2/color/image_raw</imageTopicName>
-          <cameraInfoTopicName>/cam_d2/color/camera_info</cameraInfoTopicName>
-          <depthImageTopicName>/cam_d2/depth/image_rect_raw</depthImageTopicName>
-          <depthImageCameraInfoTopicName>/cam_d2/depth/camera_info</depthImageCameraInfoTopicName>
-          <pointCloudTopicName>/cam_d2/depth/color/points</pointCloudTopicName>
-          <frameName>cam_d2_depth_link</frameName>
-          <pointCloudCutoff>0.3</pointCloudCutoff>
-          <pointCloudCutoffMax>6.0</pointCloudCutoffMax>
-          <distortionK1>0</distortionK1>
-          <distortionK2>0</distortionK2>
-          <distortionK3>0</distortionK3>
-          <distortionT1>0</distortionT1>
-          <distortionT2>0</distortionT2>
-          <CxPrime>0</CxPrime>
-          <Cx>0</Cx>
-          <Cy>0</Cy>
-          <focalLength>0</focalLength>
-          <hackBaseline>0</hackBaseline>
-        </plugin>
-      </sensor>
-  </gazebo>
-  <gazebo reference="cam_t1_pose_frame">
-    <sensor name="imu_sensor" type="imu">
-      <always_on>true</always_on>
-      <update_rate>100</update_rate>
-      <visualize>true</visualize>
-      <gravity>true</gravity>
-      <plugin filename="libgazebo_ros_imu_sensor.so" name="imu_plugin">
-        <topicName>/cam_t1/imu</topicName>
-        <bodyName>cam_t1_pose_frame</bodyName>
-        <updateRateHZ>0.0</updateRateHZ>
-        <gaussianNoise>0.002</gaussianNoise>
-        <xyzOffset>0 0 0</xyzOffset>
-        <rpyOffset>0 0 0</rpyOffset>
-        <frameName>cam_t1_pose_frame</frameName>
-        <initialOrientationAsReference>true</initialOrientationAsReference>
-      </plugin>
-      <pose>0 0 0 0 0 0</pose>
-    </sensor>
-  </gazebo>
-  </xacro:unless>
   <gazebo>
     <plugin filename="libOmniVeyorPlugin_ROS.so" name="omniveyor_simulator"/>

File: urdf/omniveyor.urdf.xacro (robot description, xacro)
@@ -2,38 +2,51 @@
 <robot name="omniveyor" xmlns:xacro="http://www.ros.org/wiki/xacro">
   <xacro:arg name="gazebo" default="false"/>
+  <!--The following arguments only takes effect in simulation.-->
   <xacro:arg name="gpu_ray_tracing" default="true"/>
-  <xacro:arg name="simulate_accurate_realsense_cameras" default="true"/>
-  <xacro:include filename="omniveyor.materials.xacro"/>
+  <xacro:arg name="has_lidar" default="true"/>
+  <xacro:arg name="has_front_d435i" default="true"/>
+  <xacro:arg name="has_rear_d435i" default="true"/>
+  <xacro:arg name="has_t265" default="true"/>
+  <xacro:arg name="simulate_full_sensor_model" default="false"/>
+  <xacro:property name="gazebo_property" value="$(arg gazebo)"/>
   <xacro:if value="$(arg gazebo)">
+    <xacro:include filename="omniveyor.materials.xacro"/>
     <!-- Gazebo Tags -->
     <!--xacro:include filename="$(find omniveyor_gazebo_world)/models/Omniveyor/omniveyor.gazebo.xacro"/-->
     <xacro:include filename="omniveyor.gazebo.xacro"/>
+    <link name="chassis">
+      <inertial>
+        <origin xyz="0 0 0.192" rpy="0 0 0"/>
+        <mass value="29.82"/>
+        <inertia ixx="1.209698" ixy="0" ixz="0"
+            iyy="1.209698" iyz="0" izz="1.910468"/>
+      </inertial>
+      <collision>
+        <origin xyz="-0.3752 0.3381 0.032" rpy="${pi/2} 0 0"/>
+        <geometry>
+          <mesh filename="package://omniveyor_common/meshes/OV_Shell.STL"
+                scale="0.001 0.001 0.001"/>
+        </geometry>
+      </collision>
+      <visual>
+        <origin xyz="-0.3752 0.3381 0.032" rpy="${pi/2} 0 0"/>
+        <geometry>
+          <mesh filename="package://omniveyor_common/meshes/OV_Shell.STL"
+                scale="0.001 0.001 0.001"/>
+        </geometry>
+        <material name="grey"/>
+      </visual>
+    </link>
+    <joint name="base_link_dummy" type="fixed">
+      <parent link="base_link" />
+      <child link="chassis" />
+      <origin xyz="0 0 0" rpy="0 0 0" />
+    </joint>
   </xacro:if>
+  <xacro:include filename="omniveyor.realsense.xacro"/>
+  <xacro:add_realsense_cameras isGazebo="$(arg gazebo)" hasFrontD435i="$(arg has_front_d435i)"
+      hasRearD435i="$(arg has_rear_d435i)" hasT265="$(arg has_t265)" useFullModel="$(arg simulate_full_sensor_model)"/>
   <!--geometric center of omniveyor (on-ground)-->
-  <link name="base_link">
-  <xacro:if value="$(arg gazebo)">
-    <inertial>
-      <origin xyz="0 0 0.192" rpy="0 0 0"/>
-      <mass value="29.82"/>
-      <inertia ixx="1.209698" ixy="0" ixz="0"
-          iyy="1.209698" iyz="0" izz="1.910468"/>
-    </inertial>
-    <collision>
-      <origin xyz="-0.3752 0.3381 0.032" rpy="${pi/2} 0 0"/>
-      <geometry>
-        <mesh filename="package://omniveyor_common/meshes/OV_Shell.STL"
-              scale="0.001 0.001 0.001"/>
-      </geometry>
-    </collision>
-    <visual>
-      <origin xyz="-0.3752 0.3381 0.032" rpy="${pi/2} 0 0"/>
-      <geometry>
-        <mesh filename="package://omniveyor_common/meshes/OV_Shell.STL"
-              scale="0.001 0.001 0.001"/>
-      </geometry>
-      <material name="grey"/>
-    </visual>
-  </xacro:if>
-  </link>
+  <link name="base_link"/>
   <!--Hokuyo 20LX-->
   <link name="laser">
@@ -70,89 +83,6 @@
     <origin xyz="0.27 0 0.10" rpy="0 0 0" />
   </joint>
-  <xacro:property name="accurateRealsense" value="$(find omniveyor_gazebo_world)" />
-  <xacro:property name="accurateRrealsensePlugin" value="$(find realsense_ros_gazebo)" />
-  <xacro:property name="gazebo_property" value="$(arg gazebo)"/>
-  <xacro:unless value="${accurateRealsense != '' and accurateRrealsensePlugin != '' and gazebo_property}">
-  <!--tracking camera-->
-  <link name="cam_t1_pose_frame">
-  <xacro:if value="$(arg gazebo)">
-    <inertial>
-      <mass value="0.2"/>
-      <inertia ixx="0.014395" ixy="0" ixz="0"
-               iyy="0.00384" iyz="0" izz="0.014136"/>
-    </inertial>
-    <collision>
-      <geometry>
-        <box size="0.008 0.13 0.02"/>
-      </geometry>
-    </collision>
-    <visual>
-      <geometry>
-        <mesh filename="package://omniveyor_common/meshes/realsense_r200.dae"/>
-      </geometry>
-    </visual>
-  </xacro:if>
-  </link>
-  <!--front depth camera-->
-  <link name="cam_d1_link">
-  <xacro:if value="$(arg gazebo)">
-    <inertial>
-      <mass value="0.2"/>
-      <inertia ixx="0.014395" ixy="0" ixz="0"
-               iyy="0.00384" iyz="0" izz="0.014136"/>
-    </inertial>
-    <collision>
-      <geometry>
-        <box size="0.02 0.13 0.02"/>
-      </geometry>
-    </collision>
-    <visual>
-      <geometry>
-        <mesh filename="package://omniveyor_common/meshes/realsense_r200.dae"/>
-      </geometry>
-    </visual>
-  </xacro:if>
-  </link>
-  <!--rear depth camera-->
-  <link name="cam_d2_link">
-  <xacro:if value="$(arg gazebo)">
-    <inertial>
-      <mass value="0.2"/>
-      <inertia ixx="0.014395" ixy="0" ixz="0"
-               iyy="0.00384" iyz="0" izz="0.014136"/>
-    </inertial>
-    <collision>
-      <geometry>
-        <box size="0.02 0.13 0.02"/>
-      </geometry>
-    </collision>
-    <visual>
-      <geometry>
-        <mesh filename="package://omniveyor_common/meshes/realsense_r200.dae"/>
-      </geometry>
-    </visual>
-  </xacro:if>
-  </link>
-  <joint name="front_t265_joint" type="fixed">
-  <!--front tracking camera connector from bottom (on-ground) center of omniveyor-->
-    <parent link="base_link" />
-    <child link="cam_t1_pose_frame" />
-    <origin xyz="0.285 -0.08 0.37" rpy="0 0 0" />
-  </joint>
-  <joint name="front_rs_joint" type="fixed">
-  <!--front depth camera connector from bottom (on-ground) center of omniveyor-->
-    <parent link="base_link" />
-    <child link="cam_d1_link" />
-    <origin xyz="0.285 0.08 0.37" rpy="0 0.04 0" />
-  </joint>
-  <joint name="rear_rs_joint" type="fixed">
-  <!--rear depth camera connector from bottom (on-ground) center of omniveyor-->
-    <parent link="base_link" />
-    <child link="cam_d2_link" />
-    <origin xyz="-0.285 -0.08 0.37" rpy="0 0.04 ${pi}" />
-  </joint>
-  </xacro:unless>
-  <xacro:if value="${accurateRealsense != '' and accurateRrealsensePlugin != '' and gazebo_property}">
+  <!--xacro:if value="${accurateRealsense != '' and accurateRrealsensePlugin != '' and gazebo_property}">
     <xacro:include filename="$(find omniveyor_gazebo_world)/launch/realsense_accurate_setup.gazebo.xacro"/>
-  </xacro:if>
+  </xacro:if-->
 </robot>
